File: PCB/hackpad.kicad_pcb (KiCad board)
At the start: 2 copper layers, 59 x 99.5 mm, 16 parts, among them SW1 SW_Push, SW10 SW_Push, SW11 SW_Push, SW12 SW_Push, SW13 RotaryEncoder_Switch, SW2 SW_Push, SW3 SW_Push, SW4 SW_Push, SW5 SW_Push, SW6 SW_Push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

Commit message: .
Parts:
- moved R1 19.0 mm to (146.5, 33.0), turned to -90 degrees
- moved R2 18.4 mm to (164.5, 46.3), turned to 180 degrees
- moved SW13 5.20 mm to (151.5, 32.4)
Routing:
- net Net-(U1-GPIO3/MOSI): track 52.5 -> 17.8 mm
- net Net-(U1-GPIO4/MISO): track 14.3 -> 38.4 mm
- net Net-(U1-VBUS): track 19.4 -> 29.6 mm
- net Net-(U1-GND): track 28.5 -> 25.3 mm
Changed lines of the file:
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@@
 	(footprint "Rotary_Encoder:RotaryEncoder_Alps_EC11E-Switch_Vertical_H20mm"
 		(layer "F.Cu")
-		(at 152.5 37.5)
+		(at 151.46 32.41)
 		(descr "Alps rotary encoder, EC11E... with switch, vertical shaft, http://www.alps.com/prod/info/E/HTML/Encoder/Incremental/EC11/EC11E15204A3.html")
 		(tags "rotary encoder")
 		(property "Reference" "SW13"
-			(at 2.8 -4.7 0)
+			(at 3.61 -1.51 0)
 			(layer "F.SilkS")
+			(hide yes)
 			(effects
 				(font
@@
 	(footprint "Resistor_THT:R_Axial_DIN0207_L6.3mm_D2.5mm_P10.16mm_Horizontal"
 		(layer "F.Cu")
-		(at 146.25 44.08 90)
+		(at 164.48 46.28 180)
 		(descr "Resistor, Axial_DIN0207 series, Axial, Horizontal, pin pitch=10.16mm, 0.25W = 1/4W, length*diameter=6.3*2.5mm^2, http://cdn-reichelt.de/documents/datenblatt/B400/1_4W%23YAG.pdf")
 		(tags "Resistor Axial_DIN0207 series Axial Horizontal pin pitch 10.16mm 0.25W = 1/4W length 6.3mm diameter 2.5mm")
 		(property "Reference" "R2"
-			(at 1.83 2.75 90)
+			(at 1.83 2.75 0)
 			(layer "F.SilkS")
 			(hide yes)
@@
 		)
 		(property "Value" "R_US"
-			(at 5.08 2.37 90)
+			(at 5.08 2.37 0)
 			(layer "F.Fab")
 			(effects
@@
 		)
 		(property "Datasheet" "~"
-			(at 0 0 90)
+			(at 0 0 0)
 			(layer "F.Fab")
 			(hide yes)
@@
 		)
 		(property "Description" "Resistor, US symbol"
-			(at 0 0 90)
+			(at 0 0 0)
 			(layer "F.Fab")
 			(hide yes)
@@
 		)
 		(fp_text user "${REFERENCE}"
-			(at 5.08 0 90)
+			(at 5.08 0 0)
 			(layer "F.Fab")
 			(effects
@@
 		)
 		(pad "1" thru_hole circle
-			(at 0 0 90)
+			(at 0 0 180)
 			(size 1.6 1.6)
 			(drill 0.8)
@@
 		)
 		(pad "2" thru_hole circle
-			(at 10.16 0 90)
+			(at 10.16 0 180)
 			(size 1.6 1.6)
 			(drill 0.8)
@@
 	(footprint "Resistor_THT:R_Axial_DIN0207_L6.3mm_D2.5mm_P10.16mm_Horizontal"
 		(layer "F.Cu")
-		(at 165.25 29.5 180)
+		(at 146.54 33.04 -90)
 		(descr "Resistor, Axial_DIN0207 series, Axial, Horizontal, pin pitch=10.16mm, 0.25W = 1/4W, length*diameter=6.3*2.5mm^2, http://cdn-reichelt.de/documents/datenblatt/B400/1_4W%23YAG.pdf")
 		(tags "Resistor Axial_DIN0207 series Axial Horizontal pin pitch 10.16mm 0.25W = 1/4W length 6.3mm diameter 2.5mm")
 		(property "Reference" "R1"
-			(at 5.08 -2.37 0)
+			(at 4.73 -2.27 90)
 			(layer "F.SilkS")
 			(effects
@@
 		)
 		(property "Value" "10K"
-			(at 5.08 2.37 0)
+			(at 5.08 2.37 90)
 			(layer "F.Fab")
 			(effects
@@
 		)
 		(property "Datasheet" "~"
-			(at 0 0 0)
+			(at 0 0 90)
 			(layer "F.Fab")
 			(hide yes)
@@
 		)
 		(property "Description" "Resistor, US symbol"
-			(at 0 0 0)
+			(at 0 0 90)
 			(layer "F.Fab")
 			(hide yes)
@@
 		(attr through_hole)
 		(fp_line
-			(start 9.12 0)
-			(end 8.35 0)
+			(start 1.04 0)
+			(end 1.81 0)
 			(stroke
 				(width 0.12)
@@
 		)
 		(fp_line
-			(start 1.04 0)
-			(end 1.81 0)
+			(start 9.12 0)
+			(end 8.35 0)
 			(stroke
 				(width 0.12)
@@
 		)
 		(fp_line
-			(start 10.16 0)
-			(end 8.23 0)
+			(start 0 0)
+			(end 1.93 0)
 			(stroke
 				(width 0.1)
@@
 		)
 		(fp_line
-			(start 0 0)
-			(end 1.93 0)
+			(start 10.16 0)
+			(end 8.23 0)
 			(stroke
 				(width 0.1)
@@
 		)
 		(fp_text user "${REFERENCE}"
-			(at 5.08 0 0)
+			(at 5.08 0 90)
 			(layer "F.Fab")
 			(effects
@@
 		)
 		(pad "1" thru_hole circle
-			(at 0 0 180)
+			(at 0 0 270)
 			(size 1.6 1.6)
 			(drill 0.8)
@@
 		)
 		(pad "2" thru_hole circle
-			(at 10.16 0 180)
+			(at 10.16 0 270)
 			(size 1.6 1.6)
 			(drill 0.8)
@@
 	)
 	(gr_text "Dustin's \nmacro\npad"
-		(at 112 35 0)
+		(at 111.01 35.31 0)
 		(layer "B.SilkS")
 		(effects
@@
 	)
 	(segment
-		(start 142.9715 29.1485)
-		(end 144.1485 29.1485)
+		(start 151.24 43.2)
+		(end 154.32 46.28)
+		(width 0.2)
+		(layer "F.Cu")
+		(net 1)
+	)
+	(segment
+		(start 140.156 31.964)
+		(end 140.156 43.23931)
 		(width 0.2)
 		(layer "F.Cu")
@@
 	)
 	(segment
-		(start 155.09 29.5)
-		(end 150.67 29.5)
+		(start 141.62 30.5)
+		(end 140.156 31.964)
 		(width 0.2)
 		(layer "F.Cu")
@@
 	)
 	(segment
-		(start 144.1485 29.1485)
-		(end 146.25 31.25)
+		(start 145.477 44.263)
+		(end 146.54 43.2)
 		(width 0.2)
 		(layer "F.Cu")
@@
 	)
 	(segment
-		(start 146.25 31.25)
-		(end 146.25 33.92)
+		(start 146.54 43.2)
+		(end 151.24 43.2)
 		(width 0.2)
 		(layer "F.Cu")
@@
 	)
 	(segment
-		(start 141.62 30.5)
-		(end 142.9715 29.1485)
+		(start 140.156 43.23931)
+		(end 141.17969 44.263)
 		(width 0.2)
 		(layer "F.Cu")
@@
 	)
 	(segment
-		(start 150.67 29.5)
-		(end 146.25 33.92)
+		(start 141.17969 44.263)
+		(end 145.477 44.263)
 		(width 0.2)
 		(layer "F.Cu")
@@
 	(segment
 		(start 140.557 37.057)
-		(end 140.557 28.70819)
+		(end 140.557 32.59969)
+		(width 0.2)
+		(layer "F.Cu")
+		(net 2)
+	)
+	(segment
+		(start 140.557 32.59969)
+		(end 141.17969 31.977)
 		(width 0.2)
 		(layer "F.Cu")
@@
 	)
 	(segment
-		(start 160.5 29.5)
-		(end 165.25 29.5)
+		(start 145.477 31.977)
+		(end 146.54 33.04)
 		(width 0.2)
 		(layer "F.Cu")
@@
 	)
 	(segment
-		(start 152.5 37.5)
-		(end 160.5 29.5)
+		(start 150.83 33.04)
+		(end 151.46 32.41)
 		(width 0.2)
 		(layer "F.Cu")
@@
 	)
 	(segment
-		(start 151.7685 36.7685)
-		(end 152.5 37.5)
+		(start 141.17969 31.977)
+		(end 145.477 31.977)
 		(width 0.2)
 		(layer "F.Cu")
@@
 	)
 	(segment
-		(start 141.17969 28.0855)
-		(end 163.8355 28.0855)
+		(start 146.54 33.04)
+		(end 150.83 33.04)
 		(width 0.2)
 		(layer "F.Cu")
@@
 	)
 	(segment
-		(start 163.8355 28.0855)
-		(end 165.25 29.5)
+		(start 164.48 46.28)
+		(end 167.261 43.499)
 		(width 0.2)
 		(layer "F.Cu")
-		(net 2)
+		(net 3)
 	)
 	(segment
-		(start 140.557 28.70819)
-		(end 141.17969 28.0855)
+		(start 167.261 43.499)
+		(end 167.261 36.871108)
 		(width 0.2)
 		(layer "F.Cu")
-		(net 2)
+		(net 3)
 	)
 	(segment
-		(start 146.25 41.75)
-		(end 145.16 40.66)
+		(start 148.21 40.66)
+		(end 141.62 40.66)
 		(width 0.2)
 		(layer "F.Cu")
@@
 	)
 	(segment
-		(start 150.92 44.08)
-		(end 152.5 42.5)
+		(start 167.261 36.871108)
+		(end 166.498892 36.109)
 		(width 0.2)
 		(layer "F.Cu")
@@
 	)
 	(segment
-		(start 145.16 40.66)
-		(end 141.62 40.66)
+		(start 166.498892 36.109)
+		(end 152.761 36.109)
 		(width 0.2)
 		(layer "F.Cu")
@@
 	)
 	(segment
-		(start 146.25 44.08)
-		(end 146.25 41.75)
+		(start 151.46 37.41)
+		(end 148.21 40.66)
 		(width 0.2)
 		(layer "F.Cu")
@@
 	)
 	(segment
-		(start 146.25 44.08)
-		(end 150.92 44.08)
+		(start 152.761 36.109)
+		(end 151.46 37.41)
 		(width 0.2)
 		(layer "F.Cu")
@@
 	)
 	(segment
-		(start 152.5 40)
-		(end 155 37.5)
+		(start 163.46 34.91)
+		(end 151.46 34.91)
 		(width 0.2)
 		(layer "F.Cu")
@@
 	)
 	(segment
-		(start 152.5 40)
-		(end 150.75 40)
+		(start 165.96 32.41)
+		(end 163.46 34.91)
 		(width 0.2)
 		(layer "F.Cu")
@@
 	)
 	(segment
-		(start 143.79 33.04)
-		(end 142.455 33.04)
+		(start 151.46 34.91)
+		(end 144.325 34.91)
 		(width 0.2)
 		(layer "F.Cu")
@@
 	)
 	(segment
-		(start 155 37.5)
-		(end 167 37.5)
-		(width 0.2)
-		(layer "F.Cu")
-		(net 11)
-	)
-	(segment
-		(start 150.75 40)
-		(end 143.79 33.04)
+		(start 144.325 34.91)
+		(end 142.455 33.04)
 		(width 0.2)
 		(layer "F.Cu")
@@
 	)
 	(segment
-		(start 143.75325 43.2)
-		(end 142.455 43.2)
-		(width 0.2)
-		(layer "F.Cu")
-		(net 12)
-	)
-	(segment
-		(start 165.25 44.25)
-		(end 151.3171 44.25)
-		(width 0.2)
-		(layer "F.Cu")
-		(net 12)
-	)
-	(segment
-		(start 146.00475 45.4515)
-		(end 143.75325 43.2)
-		(width 0.2)
-		(layer "F.Cu")
-		(net 12)
-	)
-	(segment
-		(start 150.1156 45.4515)
-		(end 146.00475 45.4515)
+		(start 165.96 37.41)
+		(end 161.54 41.83)
 		(width 0.2)
 		(layer "F.Cu")
@@
 	)
 	(segment
-		(start 167 42.5)
-		(end 165.25 44.25)
+		(start 142.99 41.83)
+		(end 141.62 43.2)
 		(width 0.2)
 		(layer "F.Cu")
@@
 	)
 	(segment
-		(start 151.3171 44.25)
-		(end 150.1156 45.4515)
+		(start 161.54 41.83)
+		(end 142.99 41.83)
 		(width 0.2)
 		(layer "F.Cu")
